File: TargetSite/TargetSite.kicad_pcb (KiCad board)
At the start: 2 copper layers, 70 x 70 mm, 24 parts, among them J1 USB_B_Micro, J10 Conn_01x02_Female, J11 Conn_01x02_Female, J12 Conn_01x02_Female, J13 Conn_01x02_Female, J2 Conn_01x02_Female, J3 Conn_01x02_Female, J4 Conn_01x02_Female, J5 Conn_01x02_Female, J6 Conn_01x02_Female, J7 Conn_01x02_Female, J8 Conn_01x02_Female, J9 Conn_01x02_Female, U1 PIC16F1459-IP

Commit message: Update TargetSite.kicad_pcb
Parts:
- moved R1 6.35 mm to (174.4, 72.8)
- moved R2 6.35 mm to (174.4, 79.2)
- moved R3 6.35 mm to (174.4, 85.5)
- moved R4 6.35 mm to (174.4, 91.9)
- moved R5 6.35 mm to (174.4, 98.2)
- moved R6 6.35 mm to (174.4, 104.6)
- moved R7 6.35 mm to (174.4, 111.0)
- moved R8 6.35 mm to (174.4, 117.3)
- moved J10 6.35 mm to (187.2, 98.2)
- moved J11 6.35 mm to (187.2, 104.6)
- moved J12 6.35 mm to (187.2, 111.0)
- moved J13 6.35 mm to (187.2, 117.3)
- moved J6 6.35 mm to (187.2, 72.8)
- moved J7 6.35 mm to (187.2, 79.2)
- moved J8 6.35 mm to (187.2, 85.5)
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Routing:
- net /D-: track 58.0 -> 40.6 mm
- net /LED_6: track 41.8 -> 26.3 mm
- net /LED_5: track 29.3 -> 19.2 mm
- net GND: track 242.8 -> 250.8 mm, vias 0 -> 2
- net /LED_8: track 31.0 -> 24.6 mm
- net /SW_3: track 16.3 -> 10.2 mm
- net /SW_2: track 17.9 -> 11.8 mm
- net /LED_4: track 24.3 -> 18.5 mm, vias 2 -> 0
- net /SW_1: track 19.5 -> 13.9 mm
- net /LED_7: track 28.6 -> 23.4 mm
- net Net-(J9-Pad1): track 0.00 -> 5.08 mm
- net Net-(J8-Pad1): track 0.00 -> 5.08 mm
- net Net-(J13-Pad1): track 0.00 -> 5.08 mm
- net Net-(J12-Pad1): track 0.00 -> 5.08 mm
- net Net-(J11-Pad1): track 0.00 -> 5.08 mm
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- added copper zone on B.Cu, net GND
- added copper zone on F.Cu, net GND

Commit message: ガーバーデータの作成、発注
Parts:
- C1: footprint Capacitor_SMD:C_Elec_3x5.4 -> Capacitor_THT:C_Disc_D3.0mm_W1.6mm_P2.50mm
- J1: footprint Connector_USB:USB_Micro-AB_Molex_47590-0001 -> Connector_USB:USB_Micro-B_Molex_47346-0001
- moved C1 1.25 mm to (163.0, 72.8)
Routing:
- net GND: track 250.8 -> 272.6 mm, vias 2 -> 16
- net unconnected-(J1-Pad6): track 0.00 -> 12.6 mm
- net /D-: track 40.6 -> 44.6 mm
- net /USB_VCC: track 31.1 -> 34.6 mm
- net /D+: track 42.3 -> 43.1 mm
Other:
- board text added: "GTech9971"
- board text added: "TargetSite 1.0"
