File: TargetSite/TargetSite.kicad_sch (KiCad schematic)
At the start: 23 parts, among them J1 USB_B_Micro, J10 Conn_01x02_Female, J11 Conn_01x02_Female, J12 Conn_01x02_Female, J13 Conn_01x02_Female, J2 Conn_01x02_Female, J3 Conn_01x02_Female, J4 Conn_01x02_Female, J5 Conn_01x02_Female, J6 Conn_01x02_Female, J7 Conn_01x02_Female, J8 Conn_01x02_Female, J9 Conn_01x02_Female, U1 PIC16F1459-IP

Commit message: PCB回路作成中
Parts:
- C1: footprint Capacitor_SMD:C_0603_1608Metric_Pad1.08x0.95mm_HandSolder -> Capacitor_SMD:C_Elec_3x5.4
- J10, J11, J12, J13, J2, J3, J4, J5, J6, J7, J8, J9: footprint (none) -> Connector_Hirose:Hirose_DF13-02P-1.25DSA_1x02_P1.25mm_Vertical
- R1, R2, R3, R4, R5, R6, R7, R8: footprint (none) -> Resistor_THT:R_Axial_DIN0204_L3.6mm_D1.6mm_P7.62mm_Horizontal

Commit message: ガーバーデータの作成、発注
Parts:
- C1: footprint Capacitor_SMD:C_Elec_3x5.4 -> Capacitor_THT:C_Disc_D3.0mm_W1.6mm_P2.50mm
- J1: footprint Connector_USB:USB_Micro-AB_Molex_47590-0001 -> Connector_USB:USB_Micro-B_Molex_47346-0001
Changed lines of the file:
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@@
     (property "Reference" "J1" (id 0) (at 34.29 44.45 0))
     (property "Value" "USB_B_Micro" (id 1) (at 34.29 46.99 0))
-    (property "Footprint" "Connector_USB:USB_Micro-AB_Molex_47590-0001" (id 2) (at 38.1 58.42 0)
+    (property "Footprint" "Connector_USB:USB_Micro-B_Molex_47346-0001" (id 2) (at 38.1 58.42 0)
       (effects (font (size 1.27 1.27)) hide)
     )
@@
     (property "Reference" "C1" (id 0) (at 130.81 52.07 90))
     (property "Value" "0.01u" (id 1) (at 130.81 54.61 90))
-    (property "Footprint" "Capacitor_SMD:C_Elec_3x5.4" (id 2) (at 134.62 58.7248 0)
+    (property "Footprint" "Capacitor_THT:C_Disc_D3.0mm_W1.6mm_P2.50mm" (id 2) (at 134.62 58.7248 0)
       (effects (font (size 1.27 1.27)) hide)
     )
@@
     )
     (path "/d917e58a-6be3-44f8-8b09-23f2c1253f7b"
-      (reference "C1") (unit 1) (value "0.01u") (footprint "Capacitor_SMD:C_Elec_3x5.4")
+      (reference "C1") (unit 1) (value "0.01u") (footprint "Capacitor_THT:C_Disc_D3.0mm_W1.6mm_P2.50mm")
     )
     (path "/42d38cba-a41c-4b30-8639-c72f3c376b19"
-      (reference "J1") (unit 1) (value "USB_B_Micro") (footprint "Connector_USB:USB_Micro-AB_Molex_47590-0001")
+      (reference "J1") (unit 1) (value "USB_B_Micro") (footprint "Connector_USB:USB_Micro-B_Molex_47346-0001")
     )
     (path "/071bccdf-8823-4317-b8f0-dcdfea517267"
